File: Piste_Blue/MOSH_ISS_THANG_STEPH_JUNJIANG.kicad_pcb (KiCad board)
At the start: 2 copper layers, 68.6 x 53.3 mm, 26 parts, among them J1 Power, J2 Digital/PWM, J3 Analog, J4 Digital/PWM, J7 LORA_STACK, Q1 IRF520, SW1 SW_SPDT, U1 LTC1050, U2 Gas_sensor, U3 MCP41100

Commit message: Add files via upload
Parts:
- moved Q1 40.9 mm to (156.5, 84.9)
- moved R8 38.3 mm to (145.8, 92.0)
- moved R7 38.0 mm to (162.0, 55.9), turned to -90 degrees
- moved R5 37.2 mm to (130.2, 54.0)
- moved R3 32.5 mm to (119.9, 72.1), turned to 180 degrees
- moved C3 28.6 mm to (119.7, 66.6)
- moved R6 28.3 mm to (140.0, 88.0), turned to 180 degrees
- moved R2 22.1 mm to (119.8, 77.0), turned to 180 degrees
- moved J7 21.6 mm to (156.0, 73.2), turned to 180 degrees
- moved C4 20.8 mm to (130.0, 72.8), turned to 90 degrees
- moved R4 18.4 mm to (130.0, 83.6), turned to 90 degrees
- moved U2 14.5 mm to (143.3, 78.9)
- moved C1 12.6 mm to (118.5, 94.0)
- moved R1 12.0 mm to (124.0, 67.0), turned to -90 degrees
- moved U1 10.0 mm to (119.5, 85.3), turned to -90 degrees
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Connections:
- J7 pad 1: TX -> RX
- J7 pad 2: RX -> TX
- J7 pad 6: +3.3V -> +3V3
- R8 pad 1: +12V -> VCC
Routing:
- net +5V: track 1.13 -> 112.5 mm, vias 0 -> 2
- net +3V3: track 0.00 -> 85.7 mm, vias 0 -> 2
- net R_potentiometer : track 0.00 -> 44.9 mm
- net Net-(U1-OUT): track 0.00 -> 44.6 mm
- net ADC1: track 1.07 -> 38.6 mm, vias 0 -> 2
- net ADC2: track 0.00 -> 32.3 mm, vias 0 -> 2
- net SW_12V: track 0.00 -> 30.3 mm
- net RX: track 0.00 -> 29.3 mm
- net CS: track 0.00 -> 29.3 mm
- net SW_1: track 0.00 -> 27.2 mm
- net IN+: track 0.00 -> 27.0 mm
- net TX: track 0.00 -> 23.7 mm
- net Net-(Q1-G): track 0.00 -> 21.2 mm
- net SCK: track 0.00 -> 20.9 mm
- net Isens: track 0.00 -> 19.6 mm
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- added copper zone on B.Cu, net GND
