File: Piste_Blue/MOSH_ISS_THANG_STEPH_JUNJIANG.kicad_sch (KiCad schematic)
At the start: 22 parts, among them J1 Power, J2 Digital/PWM, J3 Analog, J4 Digital/PWM, J7 LORA_STACK, Q1 IRF520, SW1 SW_SPDT, U1 LTC1050, U2 Gas_sensor, U3 MCP41100

Commit message: Add files via upload
Connections:
- net +12V is gone; now on net VCC: R8.1
- net +3.3V is gone; now on net +3V3: J7.6 (Pin_6)
- net RX: now also J7.1 (Pin_1); no longer J7.2 (Pin_2)
- net TX: now also J7.2 (Pin_2); no longer J7.1 (Pin_1)
Changed lines of the file:
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@@
+    (stroke (width 0) (type default))
+  )
+  (wire (pts (xy 248.92 106.045) (xy 248.92 107.95))
     (stroke (width 0) (type default))
   )
@@
     (stroke (width 0) (type default))
   )
-  (wire (pts (xy 102.87 158.75) (xy 105.41 158.75))
-    (stroke (width 0) (type default))
-  )
   (wire (pts (xy 140.97 69.85) (xy 140.97 73.66))
     (stroke (width 0) (type default))
@@
     (stroke (width 0) (type solid))
   )
-  (wire (pts (xy 102.87 156.21) (xy 105.41 156.21))
-    (stroke (width 0) (type default))
-  )
   (wire (pts (xy 248.92 55.88) (xy 248.92 58.42))
     (stroke (width 0) (type default))
@@
     (stroke (width 0) (type default))
   )
+  (wire (pts (xy 101.6 158.75) (xy 105.41 158.75))
+    (stroke (width 0) (type default))
+  )
   (wire (pts (xy 242.57 124.46) (xy 241.3 124.46))
     (stroke (width 0) (type default))
@@
     (stroke (width 0) (type solid))
   )
-  (wire (pts (xy 248.92 106.68) (xy 248.92 107.95))
-    (stroke (width 0) (type default))
-  )
   (wire (pts (xy 58.42 160.02) (xy 60.96 160.02))
     (stroke (width 0) (type default))
@@
   )
   (wire (pts (xy 207.01 55.88) (xy 218.44 55.88))
+    (stroke (width 0) (type default))
+  )
+  (wire (pts (xy 101.6 156.21) (xy 105.41 156.21))
     (stroke (width 0) (type default))
   )
@@
     )
   )
-  (global_label "RX" (shape input) (at 102.87 158.75 180) (fields_autoplaced)
+  (global_label "RX" (shape input) (at 101.6 156.21 180) (fields_autoplaced)
     (effects (font (size 1.27 1.27)) (justify right))
-    (property "Intersheetrefs" "${INTERSHEET_REFS}" (at 97.4053 158.75 0)
+    (property "Intersheetrefs" "${INTERSHEET_REFS}" (at 96.1353 156.21 0)
       (effects (font (size 1.27 1.27)) (justify right) hide)
     )
@@
     )
   )
-  (global_label "TX" (shape input) (at 102.87 156.21 180) (fields_autoplaced)
+  (global_label "TX" (shape input) (at 101.6 158.75 180) (fields_autoplaced)
     (effects (font (size 1.27 1.27)) (justify right))
-    (property "Intersheetrefs" "${INTERSHEET_REFS}" (at 97.7077 156.21 0)
+    (property "Intersheetrefs" "${INTERSHEET_REFS}" (at 96.4377 158.75 0)
       (effects (font (size 1.27 1.27)) (justify right) hide)
     )
@@
       (effects (font (size 1.27 1.27)) hide)
     )
-    (pin "2")
-    (pin "1")
+    (pin "1")
+    (pin "2")
     (instances
       (project "MOSH_ISS_THANG_STEPH_JUNJIANG"
@@
     )
   )
-  (symbol (lib_id "power:+3.3V") (at 92.71 165.1 0) (unit 1)
-    (in_bom yes) (on_board yes) (dnp no) (fields_autoplaced)
-    (property "Reference" "#PWR024" (at 92.71 168.91 0)
-      (effects (font (size 1.27 1.27)) hide)
-    )
-    (property "Value" "+3.3V" (at 92.71 160.02 0)
-      (effects (font (size 1.27 1.27)))
-    )
-    (property "Footprint" "" (at 92.71 165.1 0)
-      (effects (font (size 1.27 1.27)) hide)
-    )
-    (property "Datasheet" "" (at 92.71 165.1 0)
-      (effects (font (size 1.27 1.27)) hide)
-    )
-    (pin "1")
-    (instances
-      (project "MOSH_ISS_THANG_STEPH_JUNJIANG"
-        (path "/e63e39d7-6ac0-4ffd-8aa3-1841a4541b55"
-          (reference "#PWR024") (unit 1)
-        )
-      )
-      (project "Gas_Sensor"
-        (path "/e7501b0e-caae-4b4c-a54d-105c4777b2a1"
-          (reference "#PWR04") (unit 1)
-        )
-      )
-    )
-  )
   (symbol (lib_id "Connector_Generic:Conn_01x08") (at 110.49 163.83 0) (unit 1)
     (in_bom yes) (on_board yes) (dnp no) (fields_autoplaced)
@@
     )
     (pin "1")
-    (pin "5")
+    (pin "2")
     (pin "3")
     (pin "4")
+    (pin "5")
     (pin "6")
+    (pin "7")
     (pin "8")
-    (pin "7")
-    (pin "2")
     (instances
       (project "MOSH_ISS_THANG_STEPH_JUNJIANG"
@@
       (effects (font (size 1.27 1.27)) hide)
     )
-    (pin "2")
-    (pin "1")
+    (pin "1")
+    (pin "2")
     (instances
       (project "MOSH_ISS_THANG_STEPH_JUNJIANG"
@@
     )
   )
-  (symbol (lib_id "power:+12V") (at 248.92 106.68 0) (unit 1)
-    (in_bom yes) (on_board yes) (dnp no)
-    (property "Reference" "#PWR014" (at 248.92 110.49 0)
-      (effects (font (size 1.27 1.27)) hide)
-    )
-    (property "Value" "+12V" (at 245.11 105.41 0)
-      (effects (font (size 1.27 1.27)))
-    )
-    (property "Footprint" "" (at 248.92 106.68 0)
-      (effects (font (size 1.27 1.27)) hide)
-    )
-    (property "Datasheet" "" (at 248.92 106.68 0)
-      (effects (font (size 1.27 1.27)) hide)
-    )
-    (pin "1")
-    (instances
-      (project "MOSH_ISS_THANG_STEPH_JUNJIANG"
-        (path "/e63e39d7-6ac0-4ffd-8aa3-1841a4541b55"
-          (reference "#PWR014") (unit 1)
-        )
-      )
-      (project "Gas_Sensor"
-        (path "/e7501b0e-caae-4b4c-a54d-105c4777b2a1"
-          (reference "#PWR015") (unit 1)
-        )
-      )
-    )
-  )
   (symbol (lib_id "power:+5V") (at 217.17 31.75 0) (unit 1)
     (in_bom yes) (on_board yes) (dnp no) (fields_autoplaced)
@@
       (effects (font (size 1.27 1.27)) (justify left) hide)
     )
+    (pin "1")
+    (pin "2")
     (pin "3")
-    (pin "1")
-    (pin "2")
     (instances
       (project "MOSH_ISS_THANG_STEPH_JUNJIANG"
@@
     )
   )
+  (symbol (lib_id "power:+3V3") (at 92.71 165.1 0) (unit 1)
+    (in_bom yes) (on_board yes) (dnp no)
+    (property "Reference" "#PWR016" (at 92.71 168.91 0)
+      (effects (font (size 1.27 1.27)) hide)
+    )
+    (property "Value" "+3.3V" (at 93.091 162.052 90)
+      (effects (font (size 1.27 1.27)) (justify left))
+    )
+    (property "Footprint" "" (at 92.71 165.1 0)
+      (effects (font (size 1.27 1.27)))
+    )
+    (property "Datasheet" "" (at 92.71 165.1 0)
+      (effects (font (size 1.27 1.27)))
+    )
+    (pin "1")
+    (instances
+      (project "MOSH_ISS_THANG_STEPH_JUNJIANG"
+        (path "/e63e39d7-6ac0-4ffd-8aa3-1841a4541b55"
+          (reference "#PWR016") (unit 1)
+        )
+      )
+    )
+  )
   (symbol (lib_id "power:GND") (at 60.96 162.56 0) (unit 1)
     (in_bom yes) (on_board yes) (dnp no) (fields_autoplaced)
@@
     )
   )
+  (symbol (lib_id "power:VCC") (at 248.92 106.045 0) (unit 1)
+    (in_bom yes) (on_board yes) (dnp no)
+    (property "Reference" "#PWR014" (at 248.92 109.855 0)
+      (effects (font (size 1.27 1.27)) hide)
+    )
+    (property "Value" "VCC" (at 249.301 102.997 90)
+      (effects (font (size 1.27 1.27)) (justify left))
+    )
+    (property "Footprint" "" (at 248.92 106.045 0)
+      (effects (font (size 1.27 1.27)) hide)
+    )
+    (property "Datasheet" "" (at 248.92 106.045 0)
+      (effects (font (size 1.27 1.27)) hide)
+    )
+    (pin "1")
+    (instances
+      (project "MOSH_ISS_THANG_STEPH_JUNJIANG"
+        (path "/e63e39d7-6ac0-4ffd-8aa3-1841a4541b55"
+          (reference "#PWR014") (unit 1)
+        )
+      )
+    )
+  )
   (symbol (lib_id "Potentiometer_Digital:MCP41100") (at 48.26 157.48 0) (unit 1)
     (in_bom yes) (on_board yes) (dnp no) (fields_autoplaced)
@@
       (effects (font (size 1.27 1.27)) hide)
     )
+    (pin "1")
+    (pin "2")
+    (pin "3")
+    (pin "4")
     (pin "5")
-    (pin "2")
-    (pin "1")
     (pin "6")
-    (pin "3")
     (pin "7")
-    (pin "4")
     (pin "8")
     (instances
